File: pcb/rev.A/pc-ega-composite-daughterboard.kicad_pcb (KiCad board)
At the start: 2 copper layers, 47.5 x 43.5 mm, 45 parts, among them J1 EGA Feature Connector, U1 AD724, U2 ATF16V8, U3 AD724, Y1 3.579545 MHz, Y2 4.433619 MHz

Commit message: wip pcb rev.A
Parts:
- removed LOGO1: graphic, mygraphic:black-mage-9.6x6.5
- added JP1: Jumper_2_Open, Connector_PinHeader_2.54mm:PinHeader_1x02_P2.54mm_Vertical, F.Cu at (125.0, 119.5)
- added JP2: Jumper_2_Open, Connector_PinHeader_2.54mm:PinHeader_1x02_P2.54mm_Vertical, F.Cu at (131.2, 119.5)
- added R11: 10k, Resistor_SMD:R_0805_2012Metric_Pad1.20x1.40mm_HandSolder, F.Cu at (123.9, 115.2)
- added R12: 10k, Resistor_SMD:R_0805_2012Metric_Pad1.20x1.40mm_HandSolder, F.Cu at (123.9, 111.2)
- J1: moved to B.Cu
- R1, R3, R5: value 330 -> 390
- R13: renamed from R11; value 330 -> 390
- R15: renamed from R13; value 330 -> 390
- R17: renamed from R15; value 330 -> 390
- moved C12 3.71 mm to (132.6, 89.9)
- moved U2 2.42 mm to (126.0, 92.7)
- moved C11 2.19 mm to (126.7, 88.0), turned to -90 degrees
- moved L1 0.25 mm to (129.5, 86.3)
- turned J1 to 90 degrees
- renumbered R12 to R14, R14 to R16, R16 to R18, R17 to R19, R18 to R20, R19 to R21, R20 to R22
Connections:
- U2 pad 1: /B0_IN -> /R1_IN
- U2 pad 11: GND -> Net-(JP2-A)
- U2 pad 2: /B1_IN -> /R0_IN
- U2 pad 3: /G0_IN -> /B1_IN
- U2 pad 5: /R0_IN -> /VIN
- U2 pad 6: /R1_IN -> /B0_IN
- U2 pad 7: /VIN -> /HIN
- U2 pad 8: /HIN -> /G0_IN
- U2 pad 9: GND -> Net-(JP1-A)
Routing:
- net +5VA: track 0.00 -> 134.6 mm, vias 0 -> 5
- net /VSYNC: track 0.00 -> 62.1 mm, vias 0 -> 1
- net /HSYNC: track 0.00 -> 60.3 mm
- net /G1_IN: track 0.00 -> 56.4 mm
- net /G0_IN: track 0.00 -> 54.3 mm
- net /B1_IN: track 0.00 -> 50.3 mm
- net /HIN: track 0.00 -> 48.0 mm
- net +5V: track 0.00 -> 45.8 mm, vias 0 -> 2
- net /R0_IN: track 0.00 -> 42.1 mm
- net /PAL: track 0.00 -> 40.0 mm
- net GND: track 0.00 -> 39.9 mm, vias 0 -> 27
- net /B0_IN: track 0.00 -> 39.9 mm
- net /R1_IN: track 0.00 -> 36.1 mm
- net /VIN: track 0.00 -> 33.8 mm
- net /R1: track 0.00 -> 20.4 mm, vias 0 -> 1
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- added copper zone on B.Cu, net GND
- added copper zone on F.Cu, net GND
Other:
- board size 47.5 x 43.5 mm -> 47.5 x 44.3 mm
- board text added: "${TITLE} Rev.${REVISION}, ${COMPANY} 2023"
- board text added: "15kHz only!"
- board text added: "BOTTOM SIDE"
- board text added: "Layers: 2 Dimensions: 44.3x47.5mm Thickness: 1.6mm"
- board text added: "Min clearance: 0.2mm Min track: 0.2mm Min hole: 0.4mm Min annular ring: 0.2mm"
- board text added: "NTSC encoder"
- board text added: "PAL encoder"
- board text removed: "Layers: 2 Dimensions: 79.35x35.16mm Thickness: 1.6mm"
- board text removed: "Min clearance: 0.2mm Min track: 0.2mm Min hole: 0.3mm Min annular ring: 0.15mm"
