File: pcb/rev.A/pc-ega-composite-daughterboard.kicad_sch (KiCad schematic)
At the start: 45 parts, among them J1 EGA Feature Connector, U1 AD724, U2 ATF16V8, U3 AD724, Y1 3.579545 MHz, Y2 4.433619 MHz

Commit message: wip pcb rev.A
Parts:
- removed LOGO1: graphic, mygraphic:black-mage-9.6x6.5, symbol my:logo
- added JP1, JP2: Jumper_2_Open, Connector_PinHeader_2.54mm:PinHeader_1x02_P2.54mm_Vertical, symbol Jumper:Jumper_2_Open
- added R11, R12: 10k, Resistor_SMD:R_0805_2012Metric_Pad1.20x1.40mm_HandSolder, symbol Device:R
- R1, R3, R5: value 330 -> 390
- R13: renamed from R11; value 330 -> 390
- R15: renamed from R13; value 330 -> 390
- R17: renamed from R15; value 330 -> 390
- renumbered R12 to R14, R14 to R16, R16 to R18, R17 to R19, R18 to R20, R19 to R21, R20 to R22
Connections:
- net +5V: now also R11.1, R12.1
- net B0_IN: now also U2.6 (I6); no longer U2.1 (I1/CLK)
- net B1_IN: now also U2.3 (I3); no longer U2.2 (I2)
- net G0_IN: now also U2.8 (I8); no longer U2.3 (I3)
- net GND: now also JP1.2 (B), JP2.2 (B); no longer U2.11 (I10/~{OE}), U2.9 (I9)
- net HIN: now also U2.7 (I7); no longer U2.8 (I8)
- net R0_IN: now also U2.2 (I2); no longer U2.5 (I5)
- net R1_IN: now also U2.1 (I1/CLK); no longer U2.6 (I6)
- net VIN: now also U2.5 (I5); no longer U2.7 (I7)
- new net: JP1.1 (A), R11.2, U2.9 (I9)
- new net: JP2.1 (A), R12.2, U2.11 (I10/~{OE})
Other:
- moved on the sheet: U2
